File: spotify desk thing.kicad_sch (KiCad schematic)
At the start: 46 parts, among them J1 AudioJack3_Ground, J2 USB_C_Receptacle_USB2.0_16P, J3 DFR0669, U1 ESP32-S3-WROOM-1-N4, U2 TPA6132A2RTER, U3 PCM5242RHBR, U4 EC11E18244A5, U5 USBLC6-2SC6

Commit message: cleanup
Parts:
- renumbered C16 to C1, C11 to C10, C18 to C11, C3 to C12, C19 to C13, C4 to C14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
Connections:
- no-connect marks 7 -> 23
Other:
- moved on the sheet: BOOT1, C4
