File: pcb/spotify desk thing.kicad_pcb (KiCad board)
At the start: 2 copper layers, 113 x 50 mm, 46 parts, among them J1 USB_C_Receptacle_USB2.0_16P, J2 AudioJack3_Ground, J3 DFR0669, U1 PCM5242RHBR, U2 TPA6132A2RTER, U3 EC11E18244A5, U4 ESP32-S3-WROOM-1-N4, U5 USBLC6-2SC6

Commit message: firmware.
Parts:
- moved C18 1.90 mm to (147.6, 163.2), turned to 180 degrees
Routing:
- net Net-(C17-Pad1): track 12.6 -> 11.4 mm
Changed lines of the file:
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@@
 	(footprint "Capacitor_SMD:C_0402_1005Metric"
 		(layer "F.Cu")
-		(at 149.25 162.25)
+		(at 147.6 163.2 180)
 		(descr "Capacitor SMD 0402 (1005 Metric), square (rectangular) end terminal, IPC-7351 nominal, (Body size source: IPC-SM-782 page 76, https://www.pcb-3d.com/wordpress/wp-content/uploads/ipc-sm-782a_amendment_1_and_2.pdf), generated with kicad-footprint-generator")
 		(tags "capacitor")
 		(property "Reference" "C18"
-			(at 0 -1.16 0)
+			(at 0 1.2 0)
 			(layer "F.SilkS")
 			(effects
@@
 		)
 		(property "Part #" "TCC0402X5R105K6R3AT"
-			(at 0 0 0)
+			(at 0 0 180)
 			(unlocked yes)
 			(layer "F.Fab")
@@
 		)
 		(property "Description_1" ""
-			(at 0 0 0)
+			(at 0 0 180)
 			(unlocked yes)
 			(layer "F.Fab")
@@
 		)
 		(property "DigiKey_Part_Number" ""
-			(at 0 0 0)
+			(at 0 0 180)
 			(unlocked yes)
 			(layer "F.Fab")
@@
 		)
 		(property "MAXIMUM_PACKAGE_HEIGHT" ""
-			(at 0 0 0)
+			(at 0 0 180)
 			(unlocked yes)
 			(layer "F.Fab")
@@
 		)
 		(property "Purchase-URL" ""
-			(at 0 0 0)
+			(at 0 0 180)
 			(unlocked yes)
 			(layer "F.Fab")
@@
 		(attr smd)
 		(fp_line
-			(start -0.107836 -0.36)
-			(end 0.107836 -0.36)
+			(start -0.107836 0.36)
+			(end 0.107836 0.36)
 			(stroke
 				(width 0.12)
@@
 		)
 		(fp_line
-			(start -0.107836 0.36)
-			(end 0.107836 0.36)
+			(start -0.107836 -0.36)
+			(end 0.107836 -0.36)
 			(stroke
 				(width 0.12)
@@
 		)
 		(fp_line
-			(start -0.91 -0.46)
-			(end 0.91 -0.46)
+			(start 0.91 0.46)
+			(end -0.91 0.46)
 			(stroke
 				(width 0.05)
@@
 		)
 		(fp_line
-			(start -0.91 0.46)
-			(end -0.91 -0.46)
+			(start 0.91 -0.46)
+			(end 0.91 0.46)
 			(stroke
 				(width 0.05)
@@
 		)
 		(fp_line
-			(start 0.91 -0.46)
-			(end 0.91 0.46)
+			(start -0.91 0.46)
+			(end -0.91 -0.46)
 			(stroke
 				(width 0.05)
@@
 		)
 		(fp_line
-			(start 0.91 0.46)
-			(end -0.91 0.46)
+			(start -0.91 -0.46)
+			(end 0.91 -0.46)
 			(stroke
 				(width 0.05)
@@
 		)
 		(fp_line
-			(start -0.5 -0.25)
-			(end 0.5 -0.25)
+			(start 0.5 0.25)
+			(end -0.5 0.25)
 			(stroke
 				(width 0.1)
@@
 		)
 		(fp_line
-			(start -0.5 0.25)
-			(end -0.5 -0.25)
+			(start 0.5 -0.25)
+			(end 0.5 0.25)
 			(stroke
 				(width 0.1)
@@
 		)
 		(fp_line
-			(start 0.5 -0.25)
-			(end 0.5 0.25)
+			(start -0.5 0.25)
+			(end -0.5 -0.25)
 			(stroke
 				(width 0.1)
@@
 		)
 		(fp_line
-			(start 0.5 0.25)
-			(end -0.5 0.25)
+			(start -0.5 -0.25)
+			(end 0.5 -0.25)
 			(stroke
 				(width 0.1)
@@
 		)
 		(pad "1" smd roundrect
-			(at -0.48 0)
+			(at -0.48 0 180)
 			(size 0.56 0.62)
 			(layers "F.Cu" "F.Mask" "F.Paste")
@@
 		)
 		(pad "2" smd roundrect
-			(at 0.48 0)
+			(at 0.48 0 180)
 			(size 0.56 0.62)
 			(layers "F.Cu" "F.Mask" "F.Paste")
@@
 		(at 146.9 164.7)
 		(property "Reference" "F1"
-			(at 0.127 -1.6764 0)
+			(at -2.3 -0.1 0)
 			(layer "F.SilkS")
 			(effects
@@
 	)
 	(segment
-		(start 121.6 153.793934)
-		(end 121.6 161.6)
+		(start 101.1221 165.4779)
+		(end 100.2 166.4)
 		(width 0.2)
 		(layer "B.Cu")
@@
 	)
 	(segment
-		(start 127.454934 147.939)
-		(end 121.6 153.793934)
+		(start 121.6 161.4)
+		(end 117.5221 165.4779)
 		(width 0.2)
 		(layer "B.Cu")
@@
 	)
 	(segment
-		(start 117.7221 165.4779)
-		(end 101.1221 165.4779)
+		(start 130.2392 148.6375)
+		(end 129.5407 147.939)
 		(width 0.2)
 		(layer "B.Cu")
@@
 	)
 	(segment
-		(start 130.2392 148.6375)
-		(end 129.5407 147.939)
+		(start 127.454934 147.939)
+		(end 121.6 153.793934)
 		(width 0.2)
 		(layer "B.Cu")
@@
 	)
 	(segment
-		(start 121.6 161.6)
-		(end 117.7221 165.4779)
+		(start 117.5221 165.4779)
+		(end 101.1221 165.4779)
 		(width 0.2)
 		(layer "B.Cu")
@@
 	)
 	(segment
-		(start 101.1221 165.4779)
-		(end 100.2 166.4)
+		(start 121.6 153.793934)
+		(end 121.6 161.4)
 		(width 0.2)
 		(layer "B.Cu")
@@
 	)
 	(segment
-		(start 121.2 153.626834)
-		(end 121.2 161.4)
+		(start 98.15147 166.2)
+		(end 98.15147 165.252638)
 		(width 0.2)
 		(layer "B.Cu")
@@
 	)
 	(segment
-		(start 98.15147 166.2)
-		(end 98.15147 165.252638)
+		(start 98.934268 165)
+		(end 98.669188 164.73492)
 		(width 0.2)
 		(layer "B.Cu")
@@
 	)
 	(segment
-		(start 131.355 147.538)
-		(end 127.288834 147.538)
+		(start 117.4 165)
+		(end 98.934268 165)
 		(width 0.2)
 		(layer "B.Cu")
@@
 	)
 	(segment
-		(start 117.6 165)
-		(end 98.934268 165)
+		(start 131.355 147.538)
+		(end 127.288834 147.538)
 		(width 0.2)
 		(layer "B.Cu")
@@
 	)
 	(segment
-		(start 127.288834 147.538)
-		(end 121.2 153.626834)
+		(start 121.2 161.2)
+		(end 117.4 165)
 		(width 0.2)
 		(layer "B.Cu")
@@
 	)
 	(segment
-		(start 98.934268 165)
+		(start 98.15147 165.252638)
 		(end 98.669188 164.73492)
 		(width 0.2)
@@
 	)
 	(segment
-		(start 98.15147 165.252638)
-		(end 98.669188 164.73492)
+		(start 121.2 153.626834)
+		(end 121.2 161.2)
 		(width 0.2)
 		(layer "B.Cu")
@@
 	)
 	(segment
-		(start 121.2 161.4)
-		(end 117.6 165)
+		(start 127.288834 147.538)
+		(end 121.2 153.626834)
 		(width 0.2)
 		(layer "B.Cu")
@@
 	)
 	(segment
-		(start 126.525001 142.204234)
-		(end 126.43625 142.115483)
-		(width 0.2)
-		(layer "B.Cu")
-		(net 42)
-	)
-	(segment
-		(start 119.03 161.37)
-		(end 119.999 160.401)
+		(start 119.999 150.3661)
+		(end 119.998 150.3651)
 		(width 0.2)
 		(layer "B.Cu")
@@
 	)
 	(segment
-		(start 119.998 149.0349)
-		(end 126.4 142.6329)
+		(start 126.525001 142.474999)
+		(end 126.525001 142.204234)
 		(width 0.2)
 		(layer "B.Cu")
@@
 	)
 	(segment
-		(start 126.525001 142.474999)
-		(end 126.525001 142.204234)
+		(start 126.4 142.6)
+		(end 126.525001 142.474999)
 		(width 0.2)
 		(layer "B.Cu")
@@
 	)
 	(segment
-		(start 119.999 150.3661)
-		(end 119.998 150.3651)
+		(start 119.2629 161.37)
+		(end 119.999 160.6339)
 		(width 0.2)
 		(layer "B.Cu")
@@
 	)
 	(segment
-		(start 119.999 160.401)
-		(end 119.999 150.3661)
+		(start 126.525001 142.204234)
+		(end 126.43625 142.115483)
 		(width 0.2)
 		(layer "B.Cu")
@@
 	(segment
 		(start 117.25 161.37)
-		(end 119.03 161.37)
+		(end 119.2629 161.37)
 		(width 0.2)
 		(layer "B.Cu")
@@
 	)
 	(segment
-		(start 126.4 142.6)
-		(end 126.525001 142.474999)
+		(start 119.999 160.6339)
+		(end 119.999 150.3661)
+		(width 0.2)
+		(layer "B.Cu")
+		(net 42)
+	)
+	(segment
+		(start 119.998 149.0349)
+		(end 126.4 142.6329)
 		(width 0.2)
 		(layer "B.Cu")
@@
 	)
 	(segment
-		(start 126.187307 141.514483)
-		(end 126.685193 141.514483)
+		(start 126.685193 141.514483)
+		(end 126.885355 141.714645)
 		(width 0.2)
 		(layer "B.Cu")
@@
 	)
 	(segment
-		(start 126.885355 141.714645)
-		(end 127.714219 140.885781)
+		(start 125.83525 142.364426)
+		(end 125.83525 141.86654)
 		(width 0.2)
 		(layer "B.Cu")
@@
 	)
 	(segment
-		(start 125.968312 142.497488)
-		(end 125.83525 142.364426)
+		(start 127.714219 140.885781)
+		(end 128.218555 140.885781)
 		(width 0.2)
 		(layer "B.Cu")
@@
 	)
 	(segment
-		(start 125.83525 141.86654)
-		(end 126.187307 141.514483)
+		(start 119.2 160.6)
+		(end 119.597 160.203)
 		(width 0.2)
 		(layer "B.Cu")
@@
 	(segment
 		(start 118.4 160.6)
-		(end 119.597 159.403)
+		(end 119.2 160.6)
 		(width 0.2)
 		(layer "B.Cu")
@@
 	)
 	(segment
-		(start 119.597 159.403)
+		(start 119.597 160.203)
 		(end 119.597 148.8688)
 		(width 0.2)
@@
 	)
 	(segment
-		(start 126.685193 141.514483)
-		(end 126.885355 141.714645)
+		(start 125.968312 142.497488)
+		(end 125.83525 142.364426)
 		(width 0.2)
 		(layer "B.Cu")
@@
 	)
 	(segment
-		(start 125.83525 142.364426)
-		(end 125.83525 141.86654)
+		(start 126.885355 141.714645)
+		(end 127.714219 140.885781)
 		(width 0.2)
 		(layer "B.Cu")
@@
 	)
 	(segment
-		(start 127.714219 140.885781)
-		(end 128.218555 140.885781)
+		(start 125.83525 141.86654)
+		(end 126.187307 141.514483)
+		(width 0.2)
+		(layer "B.Cu")
+		(net 56)
+	)
+	(segment
+		(start 126.187307 141.514483)
+		(end 126.685193 141.514483)
 		(width 0.2)
 		(layer "B.Cu")
@@
 	)
 	(segment
-		(start 147.685 163.335)
-		(end 148.77 162.25)
-		(width 0.2)
+		(start 148.08 163.2)
+		(end 148.08 164.305)
+		(width 0.6)
 		(layer "F.Cu")
 		(net 64)
@@
 	(segment
 		(start 147.685 164.7)
-		(end 147.685 163.335)
-		(width 0.2)
+		(end 148.735 165.75)
+		(width 0.6)
 		(layer "F.Cu")
 		(net 64)
 	)
 	(segment
-		(start 147.685 164.7)
-		(end 148.735 165.75)
+		(start 148.08 164.305)
+		(end 147.685 164.7)
 		(width 0.6)
 		(layer "F.Cu")
@@
 		(layers "F.Cu" "B.Cu")
 		(hatch edge 0.5)
-		(connect_pads
+		(connect_pads thru_hole_only
 			(clearance 0.5)
 		)
