File: pcb/spotify desk thing.kicad_pcb (KiCad board)
At the start: 2 copper layers, 71.3 x 42 mm, 46 parts, among them J1 USB_C_Receptacle_USB2.0_16P, J2 AudioJack3_Ground, J3 ST7796, U1 PCM5242RHBR, U2 TPA6132A2RTER, U3 EC11E18244A5, U4 ESP32-S3-WROOM-1-N16R8, U5 USBLC6-2SC6

Commit message: push
Routing:
- net DGND: track 81.4 -> 66.6 mm
