File: pcb/spotify desk thing.kicad_sch (KiCad schematic)
At the start: 46 parts, among them J1 USB_C_Receptacle_USB2.0_16P, J2 AudioJack3_Ground, J3 DFR0669, U1 PCM5242RHBR, U2 TPA6132A2RTER, U3 EC11E18244A5, U4 ESP32-S3-WROOM-1-N4, U5 USBLC6-2SC6

Commit message: updated pcb with review changes
Parts:
- BOOT1, RESET1: LCSC Part # (none) -> C221784
- C1, C12, C13, C18, C4, C6, C8: LCSC Part # (none) -> C1525
- C10, C15, C7: LCSC Part # (none) -> C52923
- C11, C19: LCSC Part # (none) -> C15525
- C14, C16, C2, C5, C9: LCSC Part # (none) -> C12530
- C17: LCSC Part # (none) -> C15849
- C3: LCSC Part # (none) -> C415703
- F1: LCSC Part # (none) -> C207017
- J1: LCSC Part # (none) -> C165948
- J2: LCSC Part # (none) -> C4991872
- J3: value DFR0669 -> ST7796; footprint Connector_PinHeader_2.54mm:PinHeader_1x13_P2.54mm_Vertical -> Connector_FFC-FPC:TE_1-1734839-5_1x15-1MP_P0.5mm_Horizontal; symbol Connector:Conn_01x13_Pin -> Connector:Conn_01x14_Pin
- L1: LCSC Part # (none) -> C1043
- PS1: LCSC Part # (none) -> C40256
- R1, R3, R4, R5: LCSC Part # (none) -> C25804
- R10, R9: LCSC Part # (none) -> C25190
- R11, R7: LCSC Part # (none) -> C22859
- R12, R13: LCSC Part # (none) -> C23162
- R14, R8: LCSC Part # (none) -> C25905
- R2: LCSC (none) -> C25804
- R6: LCSC Part # (none) -> C25803
- U4: value ESP32-S3-WROOM-1-N4 -> ESP32-S3-WROOM-1-N16R8
Connections:
- net SDA: now also J3.12 (Pin_12); no longer J3.11 (Pin_11)
- net SD_CS: now also J3.14 (Pin_14); no longer J3.13 (Pin_13)
- net RST: now reaches U4.19 (IO11)
- net RST: now also J3.11 (Pin_11)
- net LCD_CS: now reaches U4.24 (IO47)
- net LCD_CS: now also J3.3 (Pin_3)
- net LCD_RST: now reaches U4.31 (IO38)
- net LCD_RST: now also J3.4 (Pin_4)
- net LCD_RS: now reaches U4.32 (IO39)
- net LCD_RS: now also J3.5 (Pin_5)
- net SCREEN_BL renamed MISO
- net SCREEN_CS renamed MOSI
- net SCREEN_DC renamed LED
- net SCREEN_MISO: no longer names the net of U4.30 (IO37)
- net SCREEN_MISO: no longer J3.5 (Pin_5)
- net SCREEN_MOSI: no longer names the net of U4.28 (IO35)
- net SCREEN_MOSI: no longer J3.4 (Pin_4)
- net SCREEN_RES renamed SCK
- net SCREEN_SCLK: no longer names the net of U4.29 (IO36)
- net SCREEN_SCLK: no longer J3.3 (Pin_3)
- net TOUCH_INT renamed INT
- net INT: now also J3.13 (Pin_13); no longer J3.12 (Pin_12)
- no-connect marks 23 -> 18

Commit message: oops forgot smtg
Parts:
- J3: footprint Connector_FFC-FPC:TE_1-1734839-5_1x15-1MP_P0.5mm_Horizontal -> Connector_FFC-FPC:TE_1-1734839-4_1x14-1MP_P0.5mm_Horizontal
Changed lines of the file:
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@@
 			)
 		)
-		(property "Footprint" "Connector_FFC-FPC:TE_1-1734839-5_1x15-1MP_P0.5mm_Horizontal"
+		(property "Footprint" "Connector_FFC-FPC:TE_1-1734839-4_1x14-1MP_P0.5mm_Horizontal"
 			(at 143.51 36.83 0)
 			(effects
